File: ISL28022_breakout_PCB/DC_Power_Monitor.kicad_pcb (KiCad board)
At the start: 2 copper layers, 59.9 x 54.9 mm, 21 parts, among them J1 DATA, J2 DATA, J3 ID_A0, J4 ID_A1, J5 PCB, J6 LOGO1, J7 LOGO2, J8 INPUT, J9 OUTPUT, U1 ISL28022

Commit message: updated PCB and instructions
Parts:
- J1, J2: footprint REInnovationFootprint:SIL-4_Grove_Labelled -> REInnovationFootprint:SIL-4_Grove_Labelled_Correct
- J3, J4: footprint REInnovationFootprint:TH_SIL_5_1mm -> REInnovationFootprint:SM_SOLDER_ID_4_WAY
- moved J3 12.3 mm to (39.8, 120.9), turned to 0 degrees
- moved J6 8.64 mm to (87.5, 121.5), turned to 270 degrees
- moved J4 7.04 mm to (45.9, 120.9), turned to 0 degrees
- moved J7 3.00 mm to (84.3, 115.8)
Connections:
- J1 pad 3: GND -> /Vcc
- J1 pad 4: /Vcc -> GND
- J2 pad 3: GND -> /Vcc
- J2 pad 4: /Vcc -> GND
- J3 pad 4: /5V -> /Vcc
- J4 pad 4: /5V -> /Vcc
- R1 pad 2: /5V -> /Vcc
- R2 pad 2: /5V -> /Vcc
Routing:
- net GND: track 168.4 -> 281.2 mm, vias 2 -> 21
- net /Ishp: track 18.2 -> 76.9 mm, vias 0 -> 26
- net /Vcc: track 30.2 -> 80.6 mm, vias 0 -> 2
- net /Ishn: track 29.3 -> 74.7 mm, vias 0 -> 18
- net Net-(J3-Pad1): track 21.0 -> 47.6 mm, vias 0 -> 2
- net /SDA: track 46.3 -> 62.8 mm, vias 0 -> 2
- net Net-(J4-Pad1): track 26.0 -> 42.4 mm
- net /SCLK: track 51.7 -> 66.4 mm, vias 1 -> 3
- net /5V: track 13.7 -> 0.00 mm
Other:
- board text added: "04/02/2021 v1.2"
- board text added: "@curiouselectric"

Commit message: updated instructions
Parts:
- moved J5 0.64 mm to (83.7, 127.2)
Routing:
- net /Ishn: track 74.7 -> 80.8 mm
- net /Ishp: track 76.9 -> 82.7 mm
- net GND: track 281.2 -> 277.4 mm

Commit message: updated
Other:
- net class Default removed
